File: flexcable/flexcable.kicad_pcb (KiCad board)
At the start: 2 copper layers, 67.8 x 133.5 mm, 6 parts

Commit message: stuff
Parts:
- added J1: Molex 200528_0400, footprints:Molex_2005280040_FPC, F.Cu at (113.0, 43.0)
- added J2: TWL_DCap_V12, footprints:FPC_Castellated_Hole, F.Cu at (174.1, 43.8)
- added J3: TWL_DCap_GND, footprints:FPC_Castellated_Hole, F.Cu at (175.0, 43.8)
- added Q1: IRFHS8342PbF, footprints:PQFN6_2X2_INF, F.Cu at (170.6, 42.4)
- added R1: 200, Resistor_SMD:R_0402_1005Metric, F.Cu at (148.2, 42.2)
- moved REF** 72.5 mm to (149.6, 81.4)
- moved REF** 72.5 mm to (151.3, 78.9)
- moved REF** 72.5 mm to (150.9, 80.9)
- moved REF** 72.5 mm to (151.1, 83.7)
- moved REF** 72.5 mm to (149.2, 78.9)
Routing:
- net /G: track 0.00 -> 1.00 mm
Other:
- board size 67.8 x 133.5 mm -> 82 x 72.1 mm
- board text removed: "see https://www.molex.com/content/dam/molex/molex-dot-com/products/automated/en-us/salesdrawingpdf/200/200528/2005280040_sd.pdf?inline"

Commit message: first fabable versions
Parts:
- removed REF** (x6): C_0201_0603Metric, Capacitor_SMD:C_0201_0603Metric
- added J4: Molex 200528_0400, footprints:Molex_2005280040_FPC, F.Cu at (187.8, 128.9)
- added J5: UTL_DCap_V12, footprints:FPC_Castellated_Hole, F.Cu at (144.6, 99.8)
- added J6: UTL_DCap_GND, footprints:FPC_Castellated_Hole, F.Cu at (144.6, 100.7)
- added J7: UTL_DCap_V12, footprints:FPC_Castellated_Hole, F.Cu at (146.4, 99.8)
- added J8: UTL_DCap_GND, footprints:FPC_Castellated_Hole, F.Cu at (146.4, 100.7)
- added Q2: IRFHS8342PbF, footprints:PQFN6_2X2_INF, F.Cu at (149.5, 97.0)
- added R2: 200, Resistor_SMD:R_0402_1005Metric, F.Cu at (152.7, 96.9)
- moved R1 26.0 mm to (163.1, 63.6)
- moved J2 21.9 mm to (169.3, 65.2)
- moved J3 21.9 mm to (170.2, 65.2)
- moved Q1 21.9 mm to (165.8, 63.7)
- moved J1 21.9 mm to (108.2, 64.3)
Connections:
- net /G renamed /G_TWL
Routing:
- net GND: track 0.00 -> 294.1 mm, vias 0 -> 25
- net /G_UTL: track 0.00 -> 70.0 mm
- net /G_TWL: track 1.00 -> 59.1 mm
- net +1V2: track 0.00 -> 17.2 mm
- net Net-(Q2-G): track 0.00 -> 2.56 mm
- net Net-(Q1-G): track 0.00 -> 2.45 mm
- added copper zone on B.Cu, net GND
Other:
- board size 82 x 72.1 mm -> 82 x 67.1 mm
- board text added: "User.4 = stiffner outline PI stiffner, T=0.3mm *total*"
- board text added: "custom layers: * User.1 = stiffner meta * User.4 = stiffner outline * User.9 = board images"
- board text removed: "conn.+ stiffner"
- board text removed: "pin 1 = GND pin 2 = V12"

Commit message: push so that i can work on this on a desktop
Parts:
- moved J4 3.48 mm to (189.6, 131.9)
Routing:
- net GND: track 294.1 -> 297.8 mm
- net /G_UTL: track 70.0 -> 71.8 mm
Other:
- board size 82 x 67.1 mm -> 83.8 x 70.1 mm
- board text added: "TODO: * larger clearance fold<->stiffner * anchor points: * TWL: 1 GPIO330? * UTL: 2 TP83+TP101? * UTL a bit longer near end? (no stiffner!) * 2mm X + 2mm Y!"

Commit message: WIP moving stuff around to make it fit
Parts:
- added H1: TWL_GPIO330, footprints:TestPointAnchor_D1.00, F.Cu at (162.4, 66.8)
- added H2: UTL_TP83_PENIRQ, footprints:TestPointAnchor_D1.00, F.Cu at (167.0, 99.8)
- added H3: UTL_TP101_HP#SP, footprints:TestPointAnchor_D1.00, F.Cu at (186.0, 98.8)
Routing:
- net GND: track 297.8 -> 20.2 mm, vias 25 -> 23
- net /G_UTL: track 71.8 -> 76.0 mm
- added copper zone on F.Cu, net GND
Other:
- outline, holes or cut-outs redrawn
- board text added: "G330"
- board text added: "TODO: * UTL a bit longer near end? (no stiffner!) * 2mm X + 3mm Y! * TODO: CHECK!"
- board text added: "TP101"
- board text added: "TP83"
- board text removed: "TODO: * larger clearance fold<->stiffner * anchor points: * TWL: 1 GPIO330? * UTL: 2 TP83+TP101? * UTL a bit longer near end? (no stiffner!) * 2mm X + 2mm Y!"
