File: flexcable/flexcable.kicad_pcb (KiCad board)
At the start: 2 copper layers, 83.8 x 70.1 mm, 15 parts, among them J1 Molex 200528_0400, J2 TWL_DCap_V12, J3 TWL_DCap_GND, J4 Molex 200528_0400, J5 UTL_DCap_V12, J6 UTL_DCap_GND, J7 UTL_DCap_V12, J8 UTL_DCap_GND, Q1 IRFHS8342PbF, Q2 IRFHS8342PbF

Commit message: version ready-ish for fabrication
Parts:
- moved J4 1.60 mm to (189.6, 130.3)
- moved H2 0.99 mm to (166.0, 99.8)
Routing:
- net /G_UTL: track 76.0 -> 74.4 mm
- net GND: vias 23 -> 21
Other:
- board size 83.8 x 70.1 mm -> 83.8 x 68.5 mm
- board text removed: "TODO: * UTL a bit longer near end? (no stiffner!) * 2mm X + 3mm Y! * TODO: CHECK!"
