File: flexcable/flexcable.kicad_sch (KiCad schematic)
At the start: 5 parts, among them J1 Molex 200528_0400, J2 TWL_DCap_V12, J3 TWL_DCap_GND, Q1 IRFHS8342PbF

Commit message: first fabable versions
Parts:
- added J4: Molex 200528_0400, footprints:Molex_2005280040_FPC, symbol Connector_Generic:Conn_01x04
- added J5, J7: UTL_DCap_V12, footprints:FPC_Castellated_Hole, symbol Connector:Conn_01x01_Socket
- added J6, J8: UTL_DCap_GND, footprints:FPC_Castellated_Hole, symbol Connector:Conn_01x01_Socket
- added Q2: IRFHS8342PbF, footprints:PQFN6_2X2_INF, symbol dsi:IRFHS8342PbF
- added R2: 200, Resistor_SMD:R_0402_1005Metric, symbol Device:R_Small_US
Connections:
- net +1V2: now also J5.1 (Pin_1), J7.1 (Pin_1), Q2.1 (D), Q2.2 (D), Q2.5 (D), Q2.6 (D), Q2.7 (D)
- net GND: now also J4.1 (Pin_1), J4.4 (Pin_4), J6.1 (Pin_1), J8.1 (Pin_1), Q2.4 (S), Q2.8 (S)
- net G renamed G_TWL
- new net: Q2.3 (G), R2.2
- new net G_UTL: J4.2 (Pin_2), J4.3 (Pin_3), R2.1
Other:
- moved on the sheet: J1, J2, J3, Q1, R1

Commit message: WIP moving stuff around to make it fit
Parts:
- added H1: TWL_GPIO330, footprints:TestPointAnchor_D1.00, symbol Mechanical:MountingHole_Pad
- added H2: UTL_TP83_PENIRQ, footprints:TestPointAnchor_D1.00, symbol Mechanical:MountingHole_Pad
- added H3: UTL_TP101_HP#SP, footprints:TestPointAnchor_D1.00, symbol Mechanical:MountingHole_Pad
- J2, J3, J5, J6, J7, J8: now left out of the parts list
Connections:
- no-connect marks 0 -> 3
Changed lines of the file:
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@@
   (junction (at 181.61 109.22) (diameter 0) (color 0 0 0 0)
   )
+  (no_connect (at 226.06 111.76))
+  (no_connect (at 226.06 119.38))
+  (no_connect (at 226.06 86.36))
   (wire (pts (xy 181.61 114.3) (xy 181.61 116.84))
     (stroke (width 0) (type default))
@@
     )
   )
+  (symbol (lib_id "Mechanical:MountingHole_Pad") (at 226.06 83.82 0) (unit 1)
+    (in_bom no) (on_board yes) (dnp no) (fields_autoplaced)
+    (property "Reference" "H1" (at 228.6 81.28 0)
+      (effects (font (size 1.27 1.27)) (justify left))
+    )
+    (property "Value" "TWL_GPIO330" (at 228.6 83.82 0)
+      (effects (font (size 1.27 1.27)) (justify left))
+    )
+    (property "Footprint" "footprints:TestPointAnchor_D1.00" (at 226.06 83.82 0)
+      (effects (font (size 1.27 1.27)) hide)
+    )
+    (property "Datasheet" "~" (at 226.06 83.82 0)
+      (effects (font (size 1.27 1.27)) hide)
+    )
+    (pin "1")
+    (instances
+      (project "flexcable"
+        (path "/e536c35a-79a7-4dc3-bafb-662c9faaf7a3"
+          (reference "H1") (unit 1)
+        )
+      )
+    )
+  )
   (symbol (lib_id "Connector:Conn_01x01_Socket") (at 189.23 114.3 0) (unit 1)
-    (in_bom yes) (on_board yes) (dnp no)
+    (in_bom no) (on_board yes) (dnp no)
     (property "Reference" "J6" (at 190.5 114.3 0)
       (effects (font (size 1.27 1.27)) (justify left))
@@
   )
   (symbol (lib_id "Connector:Conn_01x01_Socket") (at 189.23 111.76 0) (unit 1)
-    (in_bom yes) (on_board yes) (dnp no)
+    (in_bom no) (on_board yes) (dnp no)
     (property "Reference" "J5" (at 190.5 111.76 0)
       (effects (font (size 1.27 1.27)) (justify left))
@@
   )
   (symbol (lib_id "Connector:Conn_01x01_Socket") (at 189.23 81.28 0) (unit 1)
-    (in_bom yes) (on_board yes) (dnp no)
+    (in_bom no) (on_board yes) (dnp no)
     (property "Reference" "J2" (at 190.5 81.28 0)
       (effects (font (size 1.27 1.27)) (justify left))
@@
   )
   (symbol (lib_id "Connector:Conn_01x01_Socket") (at 189.23 83.82 0) (unit 1)
-    (in_bom yes) (on_board yes) (dnp no)
+    (in_bom no) (on_board yes) (dnp no)
     (property "Reference" "J3" (at 190.5 83.82 0)
       (effects (font (size 1.27 1.27)) (justify left))
@@
   )
   (symbol (lib_id "Connector:Conn_01x01_Socket") (at 189.23 116.84 0) (unit 1)
-    (in_bom yes) (on_board yes) (dnp no)
+    (in_bom no) (on_board yes) (dnp no)
     (property "Reference" "J8" (at 190.5 116.84 0)
       (effects (font (size 1.27 1.27)) (justify left))
@@
         (path "/e536c35a-79a7-4dc3-bafb-662c9faaf7a3"
           (reference "R1") (unit 1)
+        )
+      )
+    )
+  )
+  (symbol (lib_id "Mechanical:MountingHole_Pad") (at 226.06 116.84 0) (unit 1)
+    (in_bom no) (on_board yes) (dnp no) (fields_autoplaced)
+    (property "Reference" "H3" (at 228.6 114.3 0)
+      (effects (font (size 1.27 1.27)) (justify left))
+    )
+    (property "Value" "UTL_TP101_HP#SP" (at 228.6 116.84 0)
+      (effects (font (size 1.27 1.27)) (justify left))
+    )
+    (property "Footprint" "footprints:TestPointAnchor_D1.00" (at 226.06 116.84 0)
+      (effects (font (size 1.27 1.27)) hide)
+    )
+    (property "Datasheet" "~" (at 226.06 116.84 0)
+      (effects (font (size 1.27 1.27)) hide)
+    )
+    (pin "1")
+    (instances
+      (project "flexcable"
+        (path "/e536c35a-79a7-4dc3-bafb-662c9faaf7a3"
+          (reference "H3") (unit 1)
         )
       )
@@
     )
   )
+  (symbol (lib_id "Mechanical:MountingHole_Pad") (at 226.06 109.22 0) (unit 1)
+    (in_bom no) (on_board yes) (dnp no) (fields_autoplaced)
+    (property "Reference" "H2" (at 228.6 106.68 0)
+      (effects (font (size 1.27 1.27)) (justify left))
+    )
+    (property "Value" "UTL_TP83_PENIRQ" (at 228.6 109.22 0)
+      (effects (font (size 1.27 1.27)) (justify left))
+    )
+    (property "Footprint" "footprints:TestPointAnchor_D1.00" (at 226.06 109.22 0)
+      (effects (font (size 1.27 1.27)) hide)
+    )
+    (property "Datasheet" "~" (at 226.06 109.22 0)
+      (effects (font (size 1.27 1.27)) hide)
+    )
+    (pin "1")
+    (instances
+      (project "flexcable"
+        (path "/e536c35a-79a7-4dc3-bafb-662c9faaf7a3"
+          (reference "H2") (unit 1)
+        )
+      )
+    )
+  )
   (symbol (lib_id "dsi:IRFHS8342PbF") (at 147.32 111.76 0) (unit 1)
     (in_bom yes) (on_board yes) (dnp no)
@@
   )
   (symbol (lib_id "Connector:Conn_01x01_Socket") (at 189.23 109.22 0) (unit 1)
-    (in_bom yes) (on_board yes) (dnp no)
+    (in_bom no) (on_board yes) (dnp no)
     (property "Reference" "J7" (at 190.5 109.22 0)
       (effects (font (size 1.27 1.27)) (justify left))
