File: flexcable/flexcable_twl.kicad_pcb (KiCad board)
At the start: 2 copper layers, 63.3 x 5 mm, 5 parts, among them J1 Molex 200528_0400, J2 TWL_DCap_V12, J3 TWL_DCap_GND, Q1 IRFHS8342PbF

Commit message: version ready-ish for fabrication
Parts:
- added H1: TWL_GPIO330, footprints:TestPointAnchor_D1.00, F.Cu at (165.2, 96.5)
- moved R1 5.79 mm to (165.8, 93.2)
- moved J1 5.79 mm to (111.0, 94.0)
- moved J2 5.79 mm to (172.1, 94.8)
- moved J3 5.79 mm to (173.0, 94.8)
- moved Q1 5.79 mm to (168.6, 93.4)
Routing:
- net GND: track 136.0 -> 7.97 mm
- added copper zone on F.Cu, net GND
Other:
- outline, holes or cut-outs redrawn
- board text added: "G330"
- board text added: "custom layers: * User.1 = stiffner meta * User.4 = stiffner outline"
- board text removed: "custom layers: * User.1 = stiffner meta * User.4 = stiffner outline * User.9 = board images"
