File: flexcable/flexcable_utl.kicad_pcb (KiCad board)
At the start: 2 copper layers, 46.1 x 35.1 mm, 7 parts, among them J4 Molex 200528_0400, J5 UTL_DCap_V12, J6 UTL_DCap_GND, J7 UTL_DCap_V12, J8 UTL_DCap_GND, Q2 IRFHS8342PbF

Commit message: version ready-ish for fabrication
Parts:
- added H2: UTL_TP83_PENIRQ, footprints:TestPointAnchor_D1.00, F.Cu at (145.5, 85.8)
- added H3: UTL_TP101_HP#SP, footprints:TestPointAnchor_D1.00, F.Cu at (165.5, 84.8)
- moved J4 5.93 mm to (169.1, 116.3)
- moved J6 4.20 mm to (124.1, 86.7)
- moved J8 4.20 mm to (126.0, 86.7)
- moved R2 4.20 mm to (132.2, 83.0)
- moved J5 4.20 mm to (124.1, 85.8)
- moved J7 4.20 mm to (126.0, 85.8)
- moved Q2 4.20 mm to (129.0, 83.0)
Routing:
- net GND: track 157.6 -> 12.4 mm, vias 14 -> 10
- net /G_UTL: track 70.0 -> 74.3 mm
- net +1V2: track 9.21 -> 11.4 mm
- added copper zone on F.Cu, net GND
Other:
- board size 46.1 x 35.1 mm -> 47.9 x 36.5 mm
- board text added: "TP101"
- board text added: "TP83"
