File: flexcable/flexcable_fab.kicad_pcb (KiCad board)
At the start: 2 copper layers, 80.2 x 35.1 mm, 12 parts, among them J1 Molex 200528_0400, J2 TWL_DCap_V12, J3 TWL_DCap_GND, J4 Molex 200528_0400, J5 UTL_DCap_V12, J6 UTL_DCap_GND, J7 UTL_DCap_V12, J8 UTL_DCap_GND, Q1 IRFHS8342PbF, Q2 IRFHS8342PbF

Commit message: version ready-ish for fabrication
Parts:
- added H1: TWL_GPIO330, footprints:TestPointAnchor_D1.00, F.Cu at (232.0, 115.2)
- added H2: UTL_TP83_PENIRQ, footprints:TestPointAnchor_D1.00, F.Cu at (203.2, 71.7)
- added H3: UTL_TP101_HP#SP, footprints:TestPointAnchor_D1.00, F.Cu at (223.2, 70.7)
- moved J1 94.5 mm to (234.5, 61.0), turned to 0 degrees
- moved R1 43.8 mm to (235.3, 115.8), turned to 0 degrees
- moved Q1 43.2 mm to (235.1, 118.6), turned to -90 degrees
- moved J3 41.1 mm to (233.7, 123.0), turned to -135 degrees
- moved J2 41.1 mm to (233.7, 122.1), turned to -45 degrees
- moved J4 4.55 mm to (226.8, 102.3)
- moved J5 3.89 mm to (181.7, 71.8)
- moved J6 3.89 mm to (181.7, 72.7)
- moved J7 3.89 mm to (183.6, 71.8)
- moved Q2 3.89 mm to (186.7, 69.0)
- moved R2 3.89 mm to (189.9, 68.9)
- moved J8 3.89 mm to (183.6, 72.7)
Routing:
- net GND: track 293.6 -> 20.4 mm, vias 25 -> 21
- net /G_UTL: track 70.0 -> 74.3 mm
- net +1V2: track 15.2 -> 17.4 mm
- added copper zone on F.Cu, net GND
Other:
- board size 80.2 x 35.1 mm -> 55.7 x 63.3 mm
- board text added: "G330"
- board text added: "TP101"
- board text added: "TP83"
- board text added: "User.4 = stiffner outline PI stiffner, T=0.3mm *total* => 0.11mm FPC, 0.25mm stiffener stiffner on bottom side"
- board text added: "custom layers: * User.1 = stiffner meta/info * User.4 = stiffner outline/shape"
- board text removed: "2nd fold (90°)"
- board text removed: "3rd fold (90°)"
- board text removed: "4th fold (180°, diag)"
- board text removed: "User.4 = stiffner outline PI stiffner, T=0.3mm *total*"
- board text removed: "custom layers: * User.1 = stiffner meta * User.4 = stiffner outline"
- board text removed: "first fold (180°)"

Commit message: final tweaks (hopefully)
Other:
- rule pad_to_mask_clearance: 0 -> 0.1
- board text added: "JLCJLCJLCJCL"
Changed lines of the file:
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@@
   (paper "A4")
   (layers
-    (0 "F.Cu" signal)
-    (31 "B.Cu" signal)
+    (0 "F.Cu" mixed)
+    (31 "B.Cu" power)
     (32 "B.Adhes" user "B.Adhesive")
     (33 "F.Adhes" user "F.Adhesive")
@@
       (layer "B.Paste" (type "Bottom Solder Paste"))
       (layer "B.SilkS" (type "Bottom Silk Screen"))
-      (layer "F.SilkS" (type "Top Silk Screen"))
-      (layer "F.Paste" (type "Top Solder Paste"))
-      (layer "F.Mask" (type "Top Solder Mask") (thickness 0.05) (material "Dry Film") (epsilon_r 3.3) (loss_tangent 0))
-      (layer "F.Cu" (type "copper") (thickness 0.035))
-      (layer "dielectric 2" (type "core") (color "Polyimide") (thickness 0.11) (material "Polyimide") (epsilon_r 3.2) (loss_tangent 0.004))
-      (layer "B.Cu" (type "copper") (thickness 0.035))
-      (layer "B.Mask" (type "Bottom Solder Mask") (thickness 0.05) (material "Dry Film") (epsilon_r 3.3) (loss_tangent 0))
-      (layer "B.Paste" (type "Bottom Solder Paste"))
-      (layer "B.SilkS" (type "Bottom Silk Screen"))
-      (layer "F.SilkS" (type "Top Silk Screen"))
-      (layer "F.Paste" (type "Top Solder Paste"))
-      (layer "F.Mask" (type "Top Solder Mask") (thickness 0.05) (material "Dry Film") (epsilon_r 3.3) (loss_tangent 0))
-      (layer "F.Cu" (type "copper") (thickness 0.035))
-      (layer "dielectric 3" (type "core") (color "Polyimide") (thickness 0.11) (material "Polyimide") (epsilon_r 3.2) (loss_tangent 0.004))
-      (layer "B.Cu" (type "copper") (thickness 0.035))
-      (layer "B.Mask" (type "Bottom Solder Mask") (thickness 0.05) (material "Dry Film") (epsilon_r 3.3) (loss_tangent 0))
-      (layer "B.Paste" (type "Bottom Solder Paste"))
-      (layer "B.SilkS" (type "Bottom Silk Screen"))
       (copper_finish "ENIG")
       (dielectric_constraints no)
@@
       (castellated_pads yes)
     )
-    (pad_to_mask_clearance 0)
+    (pad_to_mask_clearance 0.1)
     (pcbplotparams
       (layerselection 0x02410fc_ffffffff)
@@
     (fp_arc (start 2.2 -5) (mid 2.412132 -4.912132) (end 2.5 -4.7)
       (stroke (width 0.05) (type default)) (layer "User.4"))
-    (fp_arc (start 2.512132 -2.612132) (mid 2.570711 -2.753555) (end 2.712132 -2.812132)
-      (stroke (width 0.05) (type default)) (layer "User.4"))
-    (fp_arc (start 2.570711 -3.870711) (mid 2.527351 -3.93559) (end 2.512132 -4.012132)
+    (fp_arc (start 2.512132 -2.612132) (mid 2.570711 -2.753551) (end 2.712132 -2.812132)
+      (stroke (width 0.05) (type default)) (layer "User.4"))
+    (fp_arc (start 2.570711 -3.870711) (mid 2.527339 -3.93559) (end 2.512132 -4.012132)
       (stroke (width 0.05) (type default)) (layer "User.4"))
     (fp_arc (start 2.951575 -3.635871) (mid 3.032244 -3.56212) (end 3.062132 -3.456986)
       (stroke (width 0.05) (type default)) (layer "User.4"))
-    (fp_arc (start 3.062132 -3.012132) (mid 3.003554 -2.870712) (end 2.862132 -2.812132)
+    (fp_arc (start 3.062132 -3.012132) (mid 3.003554 -2.870709) (end 2.862132 -2.812132)
       (stroke (width 0.05) (type default)) (layer "User.4"))
     (pad "1" smd roundrect (at 1.5 -3.15) (size 0.7 3.3) (layers "F.Cu" "F.Mask") (roundrect_rratio 0.25)
@@
     (fp_arc (start 2.2 -5) (mid 2.412132 -4.912132) (end 2.5 -4.7)
       (stroke (width 0.05) (type default)) (layer "User.4"))
-    (fp_arc (start 2.512132 -2.612132) (mid 2.570711 -2.753555) (end 2.712132 -2.812132)
-      (stroke (width 0.05) (type default)) (layer "User.4"))
-    (fp_arc (start 2.570711 -3.870711) (mid 2.527351 -3.93559) (end 2.512132 -4.012132)
+    (fp_arc (start 2.512132 -2.612132) (mid 2.570711 -2.753551) (end 2.712132 -2.812132)
+      (stroke (width 0.05) (type default)) (layer "User.4"))
+    (fp_arc (start 2.570711 -3.870711) (mid 2.527339 -3.93559) (end 2.512132 -4.012132)
       (stroke (width 0.05) (type default)) (layer "User.4"))
     (fp_arc (start 2.951575 -3.635871) (mid 3.032244 -3.56212) (end 3.062132 -3.456986)
       (stroke (width 0.05) (type default)) (layer "User.4"))
-    (fp_arc (start 3.062132 -3.012132) (mid 3.003554 -2.870712) (end 2.862132 -2.812132)
+    (fp_arc (start 3.062132 -3.012132) (mid 3.003554 -2.870709) (end 2.862132 -2.812132)
       (stroke (width 0.05) (type default)) (layer "User.4"))
     (pad "1" smd roundrect (at 1.5 -3.15 180) (size 0.7 3.3) (layers "F.Cu" "F.Mask") (roundrect_rratio 0.25)
@@
   (gr_arc (start 237 121.575736) (mid 236.954328 121.80535) (end 236.824264 122)
     (stroke (width 0.1) (type default)) (layer "User.4"))
-  (gr_rect (start 237 65) (end 232 85.05)
+  (gr_rect (start 232 65) (end 237 85.05)
     (stroke (width 0.15) (type default)) (fill none) (layer "User.4"))
   (gr_arc (start 183.855792 71.585591) (mid 184.675848 71.038721) (end 185.64264 70.846701)
@@
   (gr_arc (start 183.854771 72.908834) (mid 183.954614 73.62863) (end 183.34264 74.020501)
     (stroke (width 0.1) (type default)) (layer "User.4"))
-  (gr_rect (start 237 93) (end 232 104)
+  (gr_rect (start 232 93) (end 237 104)
     (stroke (width 0.15) (type default)) (fill none) (layer "User.4"))
   (gr_arc (start 202.15729 71.750684) (mid 201.564128 71.632699) (end 201.061274 71.2967)
@@
   )
   (gr_text "G330" (at 232.35 109.625 -90) (layer "F.SilkS")
+    (effects (font (size 1 1) (thickness 0.15)) (justify left bottom))
+  )
+  (gr_text "JLCJLCJLCJCL" (at 236.7 80.7 90) (layer "F.SilkS")
     (effects (font (size 1 1) (thickness 0.15)) (justify left bottom))
   )
@@
       )
     )
-  )
-  (zone (net 0) (net_name "") (layers "*.Mask") (hatch edge 0.5)
-    (connect_pads (clearance 0.5))
-    (min_thickness 0) (filled_areas_thickness no)
-    (fill yes (thermal_gap 0.5) (thermal_bridge_width 0.5))
-    (polygon
-      (pts
-        (xy -1055.841823 -1073.141823)
-        (xy -1055.841823 1072.341823)
-        (xy 1089.641823 1072.341823)
-        (xy 1089.641823 -1073.141823)
-      )
-    )
