File: wifi-interposer/power.kicad_sch (KiCad schematic)
At the start: 22 parts, among them J1 USB_C_PCB, J1 USB_C_Receptacle_USB2.0, Q4 Q_Dual_NPMOS_S1G1D2S2G2D1, SW1 SW_Push, SW2 SW_Push, U3 D1213A-02SM, U5 MIC5317-1.8YD5, U6 AP2127K-3.3, U7 USBLC6-2SC6

Commit message: add README with BOM listing
Parts:
- R3: LCSC C25744 -> C25792
Changed lines of the file:
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@@
 			)
 		)
-		(property "LCSC" "C25744"
+		(property "LCSC" "C25792"
 			(at 204.47 129.54 0)
 			(effects
