File: wifi-interposer/wifi-interposer.kicad_sch (KiCad schematic)
At the start: 33 parts, among them J1 TWL_WifiConn_Plug_TO_MAINBRD, J2 TWL_WifiConn_Rcpt_TO_WIFIBRD, J8 SOICbite, U1 RP2040, U2 W25Q16JVUXIQ, U4 W25Q16JVUXIQ, U8 PCA9306DC1, Y1 12.000 MHz, Y2 12.000MHz

Commit message: add README with BOM listing
Parts:
- C3, C4: Farnell 1758953 -> 4539081
Changed lines of the file:
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@@
 			)
 		)
-		(property "Farnell" "1758953"
+		(property "Farnell" "4539081"
 			(at 40.64 152.4 90)
 			(effects
@@
 			)
 		)
-		(property "Farnell" "1758953"
+		(property "Farnell" "4539081"
 			(at 40.64 139.7 90)
 			(effects
